File: pcb/VFDSAO.kicad_sch (KiCad schematic)
At the start: 85 parts, among them J11 USB_C_Receptacle, J12 Conn_ARM_SWD_TagConnect_TC203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, J14 SLIDE, J15 BUTT, J16 Conn_02x03_Odd_Even, Q11 AO3401A, SW11 SW_Push, U11 74AHCT1G14, U12 XC6206PxxxMR, U13 FM116B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

Commit message: RTM, pushing to germany
Parts:
- added JP13: Jumper_3_Bridged12, Jumper:SolderJumper-3_P1.3mm_Bridged12_Pad1.0x1.5mm, symbol Jumper:Jumper_3_Bridged12
- added R87: DNP, Resistor_SMD:R_0402_1005Metric, symbol Device:R
- added R88: 22K, Resistor_SMD:R_0402_1005Metric, symbol Device:R
- AE11: footprint RF_Antenna:Texas_SWRA117D_2.4GHz_Left -> modAntenna:Texas_SWRA117Dmodified
- BT11, BZ11, H15, H16, H17, H18, J14, J15, JP12, SW11: now not fitted
- C11, C12, C21, C24, C26, C28, C30, C31, C32: LCSC (none) -> C307331
- C14, C15: LCSC (none) -> C1547
- C16, C17, C20: LCSC (none) -> C52923
- C18: LCSC (none) -> C440198
- C22, C25: LCSC (none) -> C1550
- D18, D20, D22, D24: LCSC (none) -> C524054
- Q11: LCSC (none) -> C15127
- R1: renamed from 5.1K11; value R -> 5.1K; LCSC (none) -> C25905
- R11, R12, R13, R16, R17, R22: LCSC (none) -> C11702
- R14: LCSC (none) -> C25905
- R15, R18, R21, R23: LCSC (none) -> C25744
- R19: value R -> 2K; LCSC (none) -> C4109
- R25: value 190K -> 200K; LCSC (none) -> C25764
- R26: value 10K -> 22K; LCSC (none) -> C25768
- U12: LCSC (none) -> C5446
- U13: LCSC C2802264 -> C2802264
- U14: LCSC (none) -> C12044
- U15: LCSC (none) -> C5713556
Connections:
- net +24V: now also R87.1
- net +3V3: now also JP11.1 (A), JP13.1 (A); no longer JP11.3 (B)
- net +BATT: no longer C27.1, D18.2 (VDD), D20.2 (VDD), D22.2 (VDD), D24.2 (VDD)
- net 3v3_G10: now also U15.29 (PA10); no longer J11.B8 (SBU2), J12.2 (SWDIO), U15.32 (SWDIO/PA13)
- net 3v3_G11: now also R22.1, U15.37 (PA15); no longer J11.A8 (SBU1), J12.4 (SWCLK), U15.36 (SWCLK/PA14)
- net 3v3_G12: now also J11.A8 (SBU1), J12.4 (SWCLK), U15.36 (SWCLK/PA14); no longer R22.1, U15.37 (PA15)
- net 3v3_G9: now also J11.B8 (SBU2), J12.2 (SWDIO), U15.32 (SWDIO/PA13); no longer U15.29 (PA10)
- net GND: now also R88.2
- net VCC: now also JP11.3 (B), Q11.2 (S), JP13.3 (B); no longer JP11.1 (A), Q11.3 (D)
- net at R24.1: now also Q11.3 (D); no longer Q11.2 (S)
- net at R25.2, R26.1, U16.3 (FB): now also R87.2, R88.1
- new net RGB_SUP: C27.1, D18.2 (VDD), D20.2 (VDD), D22.2 (VDD), D24.2 (VDD), JP13.2 (C)
