File: pcb/anode.kicad_sch (KiCad schematic)
At the start: 4 parts, among them Q31 AO3401A

Commit message: RTM, pushing to germany
Parts:
- removed Q31: AO3401A, Package_TO_SOT_SMD:SOT-23, symbol Transistor_FET:AO3401A
- added Q71: DMC3071LVT, Package_TO_SOT_SMD:SOT-23-6, symbol Transistor_FET:DMC3071LVT
- added R86: 5.1K, Resistor_SMD:R_0402_1005Metric, symbol Device:R
- R65: LCSC (none) -> C25744
- R66: LCSC (none) -> C25741
Connections:
- net +24V: now also Q71.2 (S), R86.1
- net CTRL: now also Q71.1 (G); no longer R65.1
- net GND: now also Q71.5 (S); no longer R65.2
- net OUT: now also Q71.4 (D)
- new net: Q71.3 (G), R65.2, R86.2
- new net: Q71.6 (D), R65.1
Other:
- note added: "With a 10K, 12K divider, 24V when the NMOS is on, PMos_G = 13V, VGS = 11V When NMOS is off, PMOS_G = 24V, VGS = 0 With a 5K1, 12K, @24V NMOS on, PMOS_G = 16.8, VGS = 7.2V NMOS off, PMOS_G = 24."
- moved on the sheet: C53, R65, R66
